File: PCB/Design/cartrack.brd (EAGLE design)
At the start: 75 x 55 mm, 52 parts, among them J1 POWER_JACKPTH, Q4 12MHz, Q5 LM2941, Q6 TPS70928, U1 ATMEGA644P-20AU, X1 BU-SMA-V

Commit message: I can't remember what I have done... but it was probably important.
Routing:
- net SIM_VDD: track 43.6 -> 32.2 mm
- net GSM_PWR: track 44.6 -> 34.6 mm, vias 2 -> 1
- net +2V8: track 95.2 -> 98.8 mm
- net SIM_RST_R: track 28.4 -> 25.3 mm
- net SIM_RST: track 21.9 -> 23.6 mm
Changed lines of the file:
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@@
 </elements>
 <signals>
-<signal name="GND">
+<signal name="GND" airwireshidden="yes">
 <contactref element="U$1" pad="AGND"/>
 <contactref element="U$1" pad="GND1"/>
@@
 <via x="29" y="10.9" extent="1-16" drill="0.7"/>
 <via x="39" y="43" extent="1-16" drill="0.7"/>
-<via x="52.6" y="46.5" extent="1-16" drill="0.7"/>
 <via x="64" y="47" extent="1-16" drill="0.7"/>
-<via x="47" y="51" extent="1-16" drill="0.7"/>
-<via x="47" y="49" extent="1-16" drill="0.7"/>
+<via x="46.3" y="51" extent="1-16" drill="0.7"/>
+<via x="46.4" y="48.9" extent="1-16" drill="0.7"/>
 <via x="26" y="45" extent="1-16" drill="0.7"/>
 <via x="29" y="45" extent="1-16" drill="0.7"/>
-<via x="4" y="45" extent="1-16" drill="0.7"/>
-<via x="9" y="33" extent="1-16" drill="0.7"/>
-<via x="9" y="31" extent="1-16" drill="0.7"/>
-<via x="9" y="29" extent="1-16" drill="0.7"/>
-<via x="11" y="29" extent="1-16" drill="0.7"/>
-<via x="13" y="29" extent="1-16" drill="0.7"/>
-<via x="15" y="29" extent="1-16" drill="0.7"/>
-<via x="17" y="29" extent="1-16" drill="0.7"/>
-<via x="19" y="29" extent="1-16" drill="0.7"/>
-<via x="21" y="29" extent="1-16" drill="0.7"/>
-<via x="23" y="29" extent="1-16" drill="0.7"/>
-<via x="23" y="27" extent="1-16" drill="0.7"/>
-<via x="10" y="36" extent="1-16" drill="0.7"/>
-<via x="20" y="38" extent="1-16" drill="0.7"/>
-<via x="26" y="36" extent="1-16" drill="0.7"/>
 <via x="29" y="8" extent="1-16" drill="0.7"/>
 <via x="46" y="12" extent="1-16" drill="0.7"/>
@@
 <via x="53.4" y="27.3" extent="1-16" drill="0.7"/>
 <via x="31" y="40.4" extent="1-16" drill="0.7"/>
-<via x="2.5" y="48.2" extent="1-16" drill="0.7"/>
 <via x="24.2" y="52.8" extent="1-16" drill="0.7"/>
 <via x="64.5" y="51.5" extent="1-16" drill="0.7"/>
 <via x="34" y="27.6" extent="1-16" drill="0.7"/>
 <via x="34.2" y="29.7" extent="1-16" drill="0.7"/>
-<wire x1="47" y1="49" x2="52.6" y2="46.5" width="0" layer="19" extent="1-1"/>
+<via x="49.3" y="49.5" extent="1-16" drill="0.7"/>
+<via x="52.8" y="46.7" extent="1-16" drill="0.7"/>
+<via x="67" y="38" extent="1-16" drill="0.7"/>
+<via x="70" y="38" extent="1-16" drill="0.7"/>
+<via x="70" y="42" extent="1-16" drill="0.7"/>
+<via x="70" y="46" extent="1-16" drill="0.7"/>
 </signal>
 <signal name="+4V">
@@
 <wire x1="72.95" y1="17.1" x2="73" y2="17.15" width="1.016" layer="1"/>
 <wire x1="73" y1="17.15" x2="73" y2="22" width="1.016" layer="1"/>
-<via x="49.222" y="22" extent="1-16" drill="0.7"/>
+<via x="49.222" y="22" extent="1-16" drill="1.1"/>
 <wire x1="30.7" y1="45.55" x2="33" y2="43.25" width="0.3048" layer="1"/>
 <wire x1="33" y1="43.25" x2="33" y2="37" width="0.3048" layer="1"/>
@@
 <contactref element="Q1" pad="2"/>
 <contactref element="U$4" pad="3"/>
-<wire x1="11.05" y1="20.697" x2="8.747" y2="23" width="0.3048" layer="16"/>
-<wire x1="8.747" y1="23" x2="8" y2="23" width="0.3048" layer="16"/>
-<via x="8" y="23" extent="1-16" drill="0.7"/>
-<wire x1="8" y1="23" x2="7" y2="24" width="0.3048" layer="1"/>
-<wire x1="7" y1="24" x2="7" y2="34" width="0.3048" layer="1"/>
-<wire x1="7" y1="34" x2="4.39" y2="36.61" width="0.3048" layer="1"/>
-<wire x1="4.39" y1="36.61" x2="2.34" y2="36.61" width="0.3048" layer="1"/>
 <wire x1="2.34" y1="36.61" x2="2.35" y2="36.6" width="0.3048" layer="1"/>
-<wire x1="2.35" y1="36.6" x2="4.3" y2="36.6" width="0.3048" layer="1"/>
-<wire x1="14" y1="46" x2="14" y2="45" width="0.3048" layer="16"/>
-<wire x1="14" y1="45" x2="17" y2="42" width="0.3048" layer="16"/>
-<wire x1="17" y1="42" x2="17" y2="37" width="0.3048" layer="16"/>
-<via x="17" y="37" extent="1-16" drill="0.7"/>
-<wire x1="17" y1="37" x2="14" y2="34" width="0.3048" layer="1"/>
-<wire x1="14" y1="34" x2="7" y2="34" width="0.3048" layer="1"/>
+<wire x1="2.35" y1="36.6" x2="7.6" y2="36.6" width="0.3048" layer="1"/>
+<wire x1="11" y1="40" x2="11" y2="42" width="0.3048" layer="16"/>
+<wire x1="11" y1="42" x2="14" y2="45" width="0.3048" layer="16"/>
+<wire x1="14" y1="45" x2="14" y2="46" width="0.3048" layer="16"/>
+<wire x1="11.05" y1="20.697" x2="11.05" y2="33.15" width="0.3048" layer="16"/>
+<wire x1="11.05" y1="33.15" x2="7.6" y2="36.6" width="0.3048" layer="16"/>
+<via x="7.6" y="36.6" extent="1-16" drill="0.7"/>
+<wire x1="11" y1="40" x2="7.6" y2="36.6" width="0.3048" layer="16"/>
 </signal>
 <signal name="GSM_RX">
@@
 <wire x1="17" y1="46.15" x2="16.85" y2="46" width="0.3048" layer="16"/>
 <wire x1="16.85" y1="46" x2="15.3" y2="46" width="0.3048" layer="16"/>
-<wire x1="15.3" y1="46" x2="22" y2="39.3" width="0.3048" layer="16"/>
-<wire x1="22" y1="39.3" x2="22" y2="34" width="0.3048" layer="16"/>
-<wire x1="22" y1="34" x2="25.19" y2="30.81" width="0.3048" layer="16"/>
-<wire x1="25.19" y1="30.81" x2="30.05" y2="30.81" width="0.3048" layer="16"/>
+<wire x1="15.3" y1="46" x2="16.75" y2="44.55" width="0.3048" layer="16"/>
 <wire x1="9.44" y1="42.66" x2="9.4" y2="42.62" width="0.3048" layer="1"/>
-<wire x1="9.4" y1="42.62" x2="9.4" y2="40.1" width="0.3048" layer="1"/>
-<via x="9.4" y="40.1" extent="1-16" drill="0.7"/>
-<wire x1="9.4" y1="40.1" x2="15.5" y2="34" width="0.3048" layer="16"/>
-<wire x1="15.5" y1="34" x2="22" y2="34" width="0.3048" layer="16"/>
+<wire x1="9.44" y1="42.66" x2="9.44" y2="44.34" width="0.3048" layer="1"/>
+<wire x1="9.44" y1="44.34" x2="9.7" y2="44.6" width="0.3048" layer="1"/>
+<wire x1="9.7" y1="44.6" x2="16.7" y2="44.6" width="0.3048" layer="1"/>
+<wire x1="16.7" y1="44.6" x2="16.75" y2="44.55" width="0.3048" layer="1"/>
+<via x="16.75" y="44.55" extent="1-16" drill="0.7"/>
+<wire x1="30.05" y1="30.81" x2="16.75" y2="44.11" width="0.3048" layer="16"/>
+<wire x1="16.75" y1="44.11" x2="16.75" y2="44.55" width="0.3048" layer="16"/>
 </signal>
 <signal name="SIM_RST">
 <contactref element="U$1" pad="SIM_RST"/>
 <contactref element="R3" pad="1"/>
-<wire x1="19.1" y1="46.15" x2="19" y2="46.05" width="0.3048" layer="16"/>
-<wire x1="19" y1="46.05" x2="19" y2="44" width="0.3048" layer="16"/>
-<via x="19" y="44" extent="1-16" drill="0.7"/>
-<wire x1="19" y1="44" x2="13" y2="38" width="0.3048" layer="1"/>
-<wire x1="13" y1="38" x2="7" y2="38" width="0.3048" layer="1"/>
-<wire x1="7" y1="38" x2="5.54" y2="39.46" width="0.3048" layer="1"/>
-<wire x1="5.54" y1="39.46" x2="5.54" y2="42.66" width="0.3048" layer="1"/>
+<wire x1="5.54" y1="42.66" x2="5.54" y2="46.54" width="0.3048" layer="1"/>
+<wire x1="5.54" y1="46.54" x2="9.8" y2="50.8" width="0.3048" layer="1"/>
+<wire x1="9.8" y1="50.8" x2="12.7" y2="50.8" width="0.3048" layer="1"/>
+<wire x1="12.7" y1="50.8" x2="19.1" y2="44.4" width="0.3048" layer="1"/>
+<via x="19.1" y="44.4" extent="1-16" drill="0.7"/>
+<wire x1="19.1" y1="44.4" x2="19.1" y2="46.15" width="0.3048" layer="16"/>
 </signal>
 <signal name="SIM_CLK">
@@
 <contactref element="U$13" pad="2"/>
 <contactref element="U$4" pad="6"/>
-<wire x1="19.1" y1="47.85" x2="23" y2="43.95" width="0.3048" layer="16"/>
-<wire x1="23" y1="43.95" x2="23" y2="34" width="0.3048" layer="16"/>
-<wire x1="23" y1="34" x2="23.59" y2="33.41" width="0.3048" layer="16"/>
-<wire x1="23.59" y1="33.41" x2="30.09" y2="33.41" width="0.3048" layer="16"/>
 <wire x1="19.1" y1="47.85" x2="19" y2="47.95" width="0.3048" layer="16"/>
 <wire x1="19" y1="47.95" x2="19" y2="49" width="0.3048" layer="16"/>
@@
 <wire x1="16" y1="49" x2="15.3" y2="48.3" width="0.3048" layer="16"/>
 <wire x1="15.3" y1="48.3" x2="15.3" y2="47.9" width="0.3048" layer="16"/>
+<wire x1="30.09" y1="33.41" x2="27.9" y2="35.6" width="0.3048" layer="16"/>
+<wire x1="27.9" y1="35.6" x2="27.9" y2="36.6" width="0.3048" layer="16"/>
+<wire x1="27.9" y1="36.6" x2="22.2" y2="42.3" width="0.3048" layer="16"/>
+<wire x1="22.2" y1="42.3" x2="22.2" y2="46" width="0.3048" layer="16"/>
+<wire x1="22.2" y1="46" x2="20.35" y2="47.85" width="0.3048" layer="16"/>
+<wire x1="20.35" y1="47.85" x2="19.1" y2="47.85" width="0.3048" layer="16"/>
 </signal>
 <signal name="+2V8">
@@
 <wire x1="41.38415" y1="42.502296875" x2="40.54" y2="43.346446875" width="0.6096" layer="16"/>
 <wire x1="40.54" y1="43.346446875" x2="40.54" y2="45" width="0.6096" layer="16"/>
-<wire x1="49" y1="47" x2="49" y2="50" width="0.6096" layer="16"/>
-<wire x1="49" y1="50" x2="50.27" y2="51.27" width="0.6096" layer="16"/>
 <wire x1="50.27" y1="51.27" x2="51.46" y2="51.27" width="0.6096" layer="16"/>
 <wire x1="39.45" y1="44.8" x2="39.65" y2="45" width="0.6096" layer="16"/>
@@
 <wire x1="50.88645" y1="45" x2="52.15" y2="45" width="0.6096" layer="16"/>
 <wire x1="50.88645" y1="45" x2="50.88645" y2="45.11355" width="0.6096" layer="16"/>
-<wire x1="50.88645" y1="45.11355" x2="49" y2="47" width="0.6096" layer="16"/>
 <wire x1="41.54" y1="48.73" x2="41.54" y2="42.403225" width="0.3048" layer="1"/>
 <wire x1="41.54" y1="42.403225" x2="43" y2="40.943225" width="0.3048" layer="1"/>
@@
 <wire x1="54.8" y1="34.2" x2="51.913553125" y2="34.2" width="0.3048" layer="16"/>
 <wire x1="51.913553125" y1="34.2" x2="50.615853125" y2="35.4977" width="0.3048" layer="16"/>
+<wire x1="50.88645" y1="45.11355" x2="47.8" y2="48.2" width="0.6096" layer="16"/>
+<wire x1="47.8" y1="48.2" x2="47.8" y2="51.1" width="0.6096" layer="16"/>
+<wire x1="47.8" y1="51.1" x2="48" y2="51.3" width="0.6096" layer="16"/>
+<wire x1="48" y1="51.3" x2="51.43" y2="51.3" width="0.6096" layer="16"/>
+<wire x1="51.43" y1="51.3" x2="51.46" y2="51.27" width="0.6096" layer="16"/>
 </signal>
 <signal name="N$5">
